File: design/PTXXXX_boardname.kicad_pcb (KiCad board)
At the start: 4 copper layers, 150 x 100 mm, 13 parts

Commit message: added schematic table example (I2C Bus Table) replaced layout fabrication text with table
Other:
- board text removed: "FABRICATION =========== SUMMARY: LAYER COUNT: DESIGN RULES: IMPEDANCE CONTROL: MATERIAL: COPPER WEIGHT: FINISH: RESIST COLOUR: SILKSCREEN COLOUR: DIMENSIONS: FINISHED THICKNESS: EDGE PLATING: EDGE CONNECTORS: EDGE CHAMFERING: THIEVING/VENTING: ROHS/LEAD FREE: DRILLING: PLUGGING: OTHER NOTES:"
- board text removed: "INSTRUCTIONS: =========== MULTILAYER, SURFACE MOUNT & THROUGH HOLE 4 (2 SIGNAL & POUR, 2 SPLIT PLANE) MIN 0.20MM TRACK / 0.20MM GAP / 0.30MM DRILL 90Z DIFF PAIR, OUTER 0.20MM TRACK / 0.20MM GAP 0.40MM PLANE CLEARANCE, 0.12MM TO INNER FR4 OR EQUIVALENT, RATED TG135+ AND UL94V-0 35um OUTERS AND 17.5um INNERS ENIG GREEN WHITE 100.0MM X 150.0MM 1.6MM +/- 10% MAX OVER PLATING NOT REQUIRED NOT REQUIRED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"

Commit message: corrected layer name text to User.Eco1/2 updated titleblock dates
Other:
- board text added: "Layer Name: User.Eco1 Layer Description: Other Documentation Layer"
- board text added: "Layer Name: User.Eco2 Layer Description: Other Documentation Layer"
- board text removed: "Layer Name: Eco1.User Layer Description: Other Documentation Layer"
- board text removed: "Layer Name: Eco2.User Layer Description: Other Documentation Layer"
Changed lines of the file:
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@@
 	(title_block
 		(title "Board Name")
-		(date "2023-08-08")
+		(date "2025-12-19")
 		(rev "1.0")
 		(company "XXXX Ltd")
@@
 		)
 	)
-	(gr_text "Layer Name:          Eco1.User\nLayer Description:    Other Documentation Layer"
+	(gr_text "Layer Name:          User.Eco1\nLayer Description:    Other Documentation Layer"
 		(at 67.2 27.4 0)
 		(layer "Eco1.User")
@@
 		)
 	)
-	(gr_text "Layer Name:          Eco2.User\nLayer Description:    Other Documentation Layer"
+	(gr_text "Layer Name:          User.Eco2\nLayer Description:    Other Documentation Layer"
 		(at 67.2 27.4 0)
 		(layer "Eco2.User")
