File: design/PTXXXX_boardname.kicad_sch (KiCad schematic)
At the start: 14 parts

Commit message: add text variables example dynamic calculation & R1
Parts:
- added R1: 12k, _kb_resistors:Resistor_SMD_0603_1608m, symbol _kb_resistors:Resistor_SMD_0603_1608m
Other:
- note added: "Descriptive text about a circuit block / interface. Dynamic Calculation P_{OUT} = I^{2} * ${/be6dff3f-7b56-472d-ad92-9d283766b79e/db71de54-0981-455d-832f-a7f0dcf530bc:REFERENCE} = 30mA^{2} * ${/be6dff3f-7b56-472d-ad92-9d283766b79e/db71de54-0981-455d-832f-a7f0dcf530bc:VALUE} = @{round(pow(0.030, 2) * ${/be6dff3f-7b56-472d-ad92-9d283766b79e/db71de54-0981-455d-832f-a7f0dcf530bc:VALUE}, 2)}W"
- note removed: "Descriptive text about a circuit block / interface."
Changed lines of the file:
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@@
 	)
 	(rectangle
-		(start 74.93 40.64)
-		(end 129.54 81.28)
+		(start 35.56 31.75)
+		(end 90.17 72.39)
 		(stroke
 			(width 0)
@@
 	(text "Title"
 		(exclude_from_sim no)
-		(at 140.97 43.18 0)
+		(at 101.6 34.29 0)
 		(effects
 			(font
@@
 		)
 	)
-	(text "Descriptive text about a circuit block / interface."
+	(text "Descriptive text about a circuit block / interface.\nDynamic Calculation P_{OUT} = I^{2} * ${/be6dff3f-7b56-472d-ad92-9d283766b79e/db71de54-0981-455d-832f-a7f0dcf530bc:REFERENCE} = 30mA^{2} * ${/be6dff3f-7b56-472d-ad92-9d283766b79e/db71de54-0981-455d-832f-a7f0dcf530bc:VALUE} = @{round(pow(0.030, 2) * ${/be6dff3f-7b56-472d-ad92-9d283766b79e/db71de54-0981-455d-832f-a7f0dcf530bc:VALUE}, 2)}W"
 		(exclude_from_sim no)
-		(at 140.97 46.99 0)
+		(at 101.6 41.656 0)
 		(effects
 			(font
-				(size 1.4986 1.4986)
+				(size 1.5 1.5)
 			)
 			(justify left bottom)
@@
 	(polyline
 		(pts
-			(xy 129.54 44.45) (xy 138.43 41.91)
+			(xy 90.17 35.56) (xy 99.06 33.02)
 		)
 		(stroke
@@
 					(unit 1)
 				)
+			)
+		)
+	)
+	(symbol
+		(lib_id "_kb_resistors:Resistor_SMD_0603_1608m")
+		(at 180.34 38.1 0)
+		(unit 1)
+		(body_style 1)
+		(exclude_from_sim no)
+		(in_bom yes)
+		(on_board yes)
+		(in_pos_files yes)
+		(dnp no)
+		(fields_autoplaced yes)
+		(property "Reference" "R1"
+			(at 182.88 36.8299 0)
+			(show_name no)
+			(do_not_autoplace no)
+			(effects
+				(font
+					(size 1.27 1.27)
+				)
+				(justify left)
+			)
+		)
+		(property "Value" "12k"
+			(at 182.88 39.3699 0)
+			(show_name no)
+			(do_not_autoplace no)
+			(effects
+				(font
+					(size 1.27 1.27)
+				)
+				(justify left)
+			)
+		)
+		(property "Footprint" "_kb_resistors:Resistor_SMD_0603_1608m"
+			(at 179.197 39.37 0)
+			(hide yes)
+			(show_name no)
+			(do_not_autoplace no)
+			(effects
+				(font
+					(size 1.27 1.27)
+				)
+			)
+		)
+		(property "Datasheet" "${KIPRJMOD}\\optimised_kicad-libraries\\datasheets\\resistors\\"
+			(at 179.197 39.37 0)
+			(hide yes)
+			(show_name no)
+			(do_not_autoplace no)
+			(effects
+				(font
+					(size 1.27 1.27)
+				)
+			)
+		)
+		(property "Description" "Chip Resistor 0603 (1608m) 1% 100mW"
+			(at 180.34 38.1 0)
+			(hide yes)
+			(show_name no)
+			(do_not_autoplace no)
+			(effects
+				(font
+					(size 1.27 1.27)
+				)
+			)
+		)
+		(property "Manufacturer1" "ANY"
+			(at 180.34 38.1 0)
+			(hide yes)
+			(show_name no)
+			(do_not_autoplace no)
+			(effects
+				(font
+					(size 1.27 1.27)
+				)
+			)
+		)
+		(property "MPN1" "As Appropriate"
+			(at 180.34 38.1 0)
+			(hide yes)
+			(show_name no)
+			(do_not_autoplace no)
+			(effects
+				(font
+					(size 1.27 1.27)
+				)
+			)
+		)
+		(property "Manufacturer2" " "
+			(at 180.34 38.1 0)
+			(hide yes)
+			(show_name no)
+			(do_not_autoplace no)
+			(effects
+				(font
+					(size 1.27 1.27)
+				)
+			)
+		)
+		(property "MPN2" " "
+			(at 180.34 38.1 0)
+			(hide yes)
+			(show_name no)
+			(do_not_autoplace no)
+			(effects
+				(font
+					(size 1.27 1.27)
+				)
+			)
+		)
+		(property "Vendor1" " "
+			(at 180.34 38.1 0)
+			(hide yes)
+			(show_name no)
+			(do_not_autoplace no)
+			(effects
+				(font
+					(size 1.27 1.27)
+				)
+			)
+		)
+		(property "SKU1" " "
+			(at 180.34 38.1 0)
+			(hide yes)
+			(show_name no)
+			(do_not_autoplace no)
+			(effects
+				(font
+					(size 1.27 1.27)
+				)
+			)
+		)
+		(property "Vendor2" " "
+			(at 180.34 38.1 0)
+			(hide yes)
+			(show_name no)
+			(do_not_autoplace no)
+			(effects
+				(font
+					(size 1.27 1.27)
+				)
+			)
+		)
+		(property "SKU2" " "
+			(at 180.34 38.1 0)
+			(hide yes)
+			(show_name no)
+			(do_not_autoplace no)
+			(effects
+				(font
+					(size 1.27 1.27)
+				)
+			)
+		)
+		(pin "1"
+		)
+		(pin "2"
+		)
+		(instances
+			(project "PTXXXX_boardname"
+				(path "/be6dff3f-7b56-472d-ad92-9d283766b79e"
+					(reference "R1")
+					(unit 1)
+				)

Commit message: added board name title text added variant name title text rename top sheet to root
Other:
- note added: "@{if("${VARIANT}"=="", "${TITLE}", "${TITLE} (Variant: ${VARIANT}, ${VARIANT_DESC})")}"
- note added: "Descriptive text about the circuit board."
- moved on the sheet: R1
Changed lines of the file:
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@@
 	)
 	(rectangle
-		(start 35.56 31.75)
-		(end 90.17 72.39)
+		(start 140.97 33.02)
+		(end 170.18 58.42)
 		(stroke
 			(width 0)
@@
 	(text "Title"
 		(exclude_from_sim no)
-		(at 101.6 34.29 0)
+		(at 181.61 35.56 0)
 		(effects
 			(font
@@
 		)
 	)
+	(text "Descriptive text about the circuit board."
+		(exclude_from_sim no)
+		(at 36.322 38.1 0)
+		(effects
+			(font
+				(size 1.5 1.5)
+			)
+			(justify left top)
+		)
+	)
 	(text "Descriptive text about a circuit block / interface.\nDynamic Calculation P_{OUT} = I^{2} * ${/be6dff3f-7b56-472d-ad92-9d283766b79e/db71de54-0981-455d-832f-a7f0dcf530bc:REFERENCE} = 30mA^{2} * ${/be6dff3f-7b56-472d-ad92-9d283766b79e/db71de54-0981-455d-832f-a7f0dcf530bc:VALUE} = @{round(pow(0.030, 2) * ${/be6dff3f-7b56-472d-ad92-9d283766b79e/db71de54-0981-455d-832f-a7f0dcf530bc:VALUE}, 2)}W"
 		(exclude_from_sim no)
-		(at 101.6 41.656 0)
+		(at 181.61 37.338 0)
 		(effects
 			(font
 				(size 1.5 1.5)
 			)
+			(justify left top)
+		)
+	)
+	(text "@{if(\"${VARIANT}\"==\"\", \"${TITLE}\", \"${TITLE} (Variant: ${VARIANT}, ${VARIANT_DESC})\")}"
+		(exclude_from_sim no)
+		(at 36.322 36.322 0)
+		(effects
+			(font
+				(size 2.0066 2.0066)
+				(thickness 0.4013)
+				(bold yes)
+			)
 			(justify left bottom)
 		)
@@
 	(polyline
 		(pts
-			(xy 90.17 35.56) (xy 99.06 33.02)
+			(xy 170.18 36.83) (xy 179.07 34.29)
 		)
 		(stroke
@@
 	(symbol
 		(lib_id "_kb_resistors:Resistor_SMD_0603_1608m")
-		(at 180.34 38.1 0)
+		(at 260.35 39.37 0)
 		(unit 1)
 		(body_style 1)
@@
 		(fields_autoplaced yes)
 		(property "Reference" "R1"
-			(at 182.88 36.8299 0)
+			(at 262.89 38.0999 0)
 			(show_name no)
 			(do_not_autoplace no)
@@
 		)
 		(property "Value" "12k"
-			(at 182.88 39.3699 0)
+			(at 262.89 40.6399 0)
 			(show_name no)
 			(do_not_autoplace no)
@@
 		)
 		(property "Footprint" "_kb_resistors:Resistor_SMD_0603_1608m"
-			(at 179.197 39.37 0)
+			(at 259.207 40.64 0)
 			(hide yes)
 			(show_name no)
@@
 		)
 		(property "Datasheet" "${KIPRJMOD}\\optimised_kicad-libraries\\datasheets\\resistors\\"
-			(at 179.197 39.37 0)
+			(at 259.207 40.64 0)
 			(hide yes)
 			(show_name no)
@@
 		)
 		(property "Description" "Chip Resistor 0603 (1608m) 1% 100mW"
-			(at 180.34 38.1 0)
+			(at 260.35 39.37 0)
 			(hide yes)
 			(show_name no)
@@
 		)
 		(property "Manufacturer1" "ANY"
-			(at 180.34 38.1 0)
+			(at 260.35 39.37 0)
 			(hide yes)
 			(show_name no)
@@
 		)
 		(property "MPN1" "As Appropriate"
-			(at 180.34 38.1 0)
+			(at 260.35 39.37 0)
 			(hide yes)
 			(show_name no)
@@
 		)
 		(property "Manufacturer2" " "
-			(at 180.34 38.1 0)
+			(at 260.35 39.37 0)
 			(hide yes)
 			(show_name no)
@@
 		)
 		(property "MPN2" " "
-			(at 180.34 38.1 0)
+			(at 260.35 39.37 0)
 			(hide yes)
 			(show_name no)
@@
 		)
 		(property "Vendor1" " "
-			(at 180.34 38.1 0)
+			(at 260.35 39.37 0)
 			(hide yes)
 			(show_name no)
@@
 		)
 		(property "SKU1" " "
-			(at 180.34 38.1 0)
+			(at 260.35 39.37 0)
 			(hide yes)
 			(show_name no)
@@
 		)
 		(property "Vendor2" " "
-			(at 180.34 38.1 0)
+			(at 260.35 39.37 0)
 			(hide yes)
 			(show_name no)
@@
 		)
 		(property "SKU2" " "
-			(at 180.34 38.1 0)
+			(at 260.35 39.37 0)
 			(hide yes)
 			(show_name no)
